File: usb_power.kicad_sch (KiCad schematic)
At the start: 17 parts, among them J1 GT-USB-7010ASV, Q1 AO3401A, SW1 PCM12, U1 H5VU25UC, U2 AMS1117-3.3

Commit message: Rev.2 (260322)
Parts:
- added D3: KT-0603R, LED_SMD:LED_0603_1608Metric, symbol Device:LED
- added R7: 220, Resistor_SMD:R_0402_1005Metric, symbol Device:R
- C1, C2: LCSC (none) -> C19702
- C3: LCSC (none) -> C7171
- D1: LCSC (none) -> C20615804
- D2: LCSC (none) -> C2297
- F1: LCSC (none) -> C6165191
- J1: LCSC (none) -> C2988369
- Q1: LCSC (none) -> C15127
- R1, R2: LCSC (none) -> C25905
- R3: LCSC (none) -> C25741
- R4: LCSC (none) -> C25744
- R5: LCSC (none) -> C25756
- R6: value 100 -> 2.2k; footprint Harucom_Board:R_0402_1005Metric_Pad0.566x0.54mm -> Resistor_SMD:R_0402_1005Metric; LCSC (none) -> C25879
- SW1: value PCM12 -> SK-12; footprint Button_Switch_SMD:SW_SPDT_PCM12 -> Harucom_Board:SW_Slide_SPDT_Angled_SK_12D11VG3; now not fitted
- U1: symbol Hakodate_Board:H5VU25UC -> Harucom_Board:H5VU25UC; LCSC (none) -> C20615800
- U2: LCSC (none) -> C6186
Connections:
- net GND: now also R3.2, D3.1 (K); no longer SW1.1 (A)
- net at Q1.1 (G), SW1.2 (B): now also R3.1; no longer R3.2
- net at C1.1, D1.1 (A1), F1.2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: now also SW1.1 (A); no longer R3.1
- net LED renamed LED_G
- new net: D3.2 (A), R7.2
- new net LED_R: R7.1
Other:
- moved on the sheet: D2, R3, R6

Commit message: Rev. 2B: Change PSRAM package from SOP-8 to USON-8L.
Parts:
- SW1: now left out of the parts list
Changed lines of the file:
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@@
 	(title_block
 		(title "Harucom-board")
-		(date "2026-03-22")
-		(rev "2")
+		(date "2026-03-23")
+		(rev "2B")
 		(comment 1 "https://github.com/harukasan/harucom-board/")
 		(comment 2 "SPDX-License-Identifier: CERN-OHL-P-2.0")
@@
 		(unit 1)
 		(exclude_from_sim no)
-		(in_bom yes)
+		(in_bom no)
 		(on_board yes)
 		(dnp yes)
